Commit message: update limits to real arm, add real joint-state bridge

File: src/robot_drive_by_moveit2/src/my_robot_description/urdf/arm.xacro (robot description, xacro)
@@ -146,6 +146,5 @@
         <limit effort="2.45" velocity="1.0" lower="-0.785398" upper="1.5708" />
     </joint>
-    <!-- joint3 - elbow pitch, about Y. Initial at 0deg (link vertical to
-         the ground), range +-110deg -->
+    <!-- joint3 - elbow pitch, about Y. Initial at 0deg (vertical), range +-90deg -->
     <joint name="joint3" type="revolute">
         <parent link="arm_link" />
@@ -153,5 +152,5 @@
         <origin xyz="0 0 0.118" rpy="0 0 0" />
         <axis xyz="0 1 0" />
-        <limit effort="2.45" velocity="1.0" lower="-1.91986" upper="1.91986" />
+        <limit effort="2.45" velocity="1.0" lower="-1.5708" upper="1.5708" />
     </joint>
     <!-- joint4 - wrist pitch, about Y.

File: src/robot_drive_by_moveit2/src/my_robot_description/urdf/my_robot.ros2_control.xacro (robot description, xacro)
@@ -15,6 +15,5 @@
           <command_interface name="position"/>
           <state_interface name="position">
-            <!-- initial -45deg -->
-            <param name="initial_value">-0.785398</param>
+            <param name="initial_value">0.0</param>
           </state_interface>
       </joint>
@@ -28,6 +27,5 @@
           <command_interface name="position"/>
           <state_interface name="position">
-            <!-- initial +90deg -->
-            <param name="initial_value">1.5708</param>
+            <param name="initial_value">0.0</param>
           </state_interface>
       </joint>
@@ -35,6 +33,5 @@
           <command_interface name="position"/>
           <state_interface name="position">
-            <!-- initial +90deg -->
-            <param name="initial_value">1.5708</param>
+            <param name="initial_value">0.0</param>
           </state_interface>
       </joint>

Commit message: Match URDF/simulation to the real 5-DOF arm and add calibration tools
Description and MoveIt config:

- arm.xacro: joint1/joint5 continuous -> revolute (+-135 deg) so MoveIt and RViz expose a joint slider, matching the ZP25S 270 deg travel

- arm.xacro: joint5 -> tool_link shortened from 130 mm to the measured 30 mm (wrist_hand 20 mm + hand_tool 10 mm)

- gripper.xacro: rebuilt for the real gripper (80x20x20 mm palm, 10x20x80 mm fingers, 80 mm opening, 40 mm per-finger travel, master 0.0 open -> 0.04 closed)

- my_robot.srdf: gripper_closed 0.06 -> 0.04

- CMakeLists.txt: install the mujoco directory

Simulation:

- mujoco/my_robot.xml: 7-DOF MJCF with URDF-matching limits, mimic equality constraint, 6 position actuators and home/ready keyframes. contype/conaffinity bitmasks keep the overlapping URDF collision boxes from locking the joints

- mujoco/demo.py: headless demo driven by simulated time so it stays correct at high speedup

Camera calibration and hand-eye tooling:

- tools/make_checkerboard.py + printable A4 8x6 20 mm checkerboard

- tools/check_camera.py: verify camera_info and image topics

- tools/tag_pose.py: AprilTag 36h11 6-DOF pose from a single tag (IPPE_SQUARE)

- tools/hand_eye_calibrate.py: eye-to-hand AX=ZB calibration, passes inverted robot poses to cv2.calibrateHandEye and returns T_base_cam

- tools/test_tag_pose.py, tools/test_handeye_solve.py: self-checks, both pass on OpenCV 4.5.4

Other:

- my_robot_commander_cpp/scripts/servo_scan.py: probe the ZP25S bus for servo IDs

- .gitignore: ignore build/ install/ log/ .vscode/ .history/ __pycache__/

File: src/robot_drive_by_moveit2/src/my_robot_description/urdf/arm.xacro (robot description, xacro)
@@ -111,5 +111,6 @@
     </link>
     <!-- hand_link - short fixed mount where the gripper attaches.
-         joint5 -> tool_link total = 0.11 + 0.02 = 0.13 (130mm) -->
+         joint5 -> tool_link total = 0.02 + 0.01 = 0.03 (30mm measured from
+         the servo output shaft face to the gripper base plate) -->
     <link name="hand_link">
         <visual>
@@ -129,10 +130,13 @@
     <!-- tool_link - gripper mounting frame (gripper attaches here) -->
     <link name="tool_link" />
-    <!-- joint1 - base yaw, rotation about vertical Z, continuous 360deg -->
-    <joint name="joint1" type="continuous">
+    <!-- joint1 - base yaw, about vertical Z.
+         Revolute (not continuous) so MoveIt/RViz exposes a joint slider.
+         Range +-135deg matches the ZP25S 270deg travel. -->
+    <joint name="joint1" type="revolute">
         <parent link="base_link" />
         <child link="shoulder_link" />
         <origin xyz="0 0 0" rpy="0 0 0" />
         <axis xyz="0 0 1" />
+        <limit effort="2.45" velocity="1.0" lower="-2.35619" upper="2.35619" />
     </joint>
     <!-- joint2 - shoulder pitch, about Y.
@@ -164,24 +168,27 @@
         <limit effort="2.45" velocity="1.0" lower="-1.5708" upper="1.5708" />
     </joint>
-    <!-- joint5 - wrist roll, about the arm axis Z, continuous 360deg
-         (NOTE - was Y pitch in the old model; corrected to Z roll) -->
-    <joint name="joint5" type="continuous">
+    <!-- joint5 - wrist roll, about the arm axis Z.
+         Revolute (not continuous) so MoveIt/RViz exposes a joint slider.
+         Range +-135deg matches the ZP25S 270deg travel. -->
+    <joint name="joint5" type="revolute">
         <parent link="forearm_link" />
         <child link="wrist_link" />
         <origin xyz="0 0 0.031" rpy="0 0 0" />
         <axis xyz="0 0 1" />
+        <limit effort="2.45" velocity="1.0" lower="-2.35619" upper="2.35619" />
     </joint>
-    <!-- wrist_hand_joint - fixed, wrist -> hand, 110mm (part of the 130mm) -->
+    <!-- wrist_hand_joint - fixed, wrist -> hand, 20mm of the 30mm gap -->
     <joint name="wrist_hand_joint" type="fixed">
         <parent link="wrist_link" />
         <child link="hand_link" />
-        <origin xyz="0 0 0.11" rpy="0 0 0" />
+        <origin xyz="0 0 0.02" rpy="0 0 0" />
     </joint>
-    <!-- hand_tool_joint - fixed, hand -> tool (gripper mount), 20mm.
-         joint5 -> tool_link = 0.11 + 0.02 = 0.13 (130mm to the gripper) -->
+    <!-- hand_tool_joint - fixed, hand -> tool (gripper mounting face), 10mm.
+         joint5 -> tool_link = 0.02 + 0.01 = 0.03 (30mm, servo shaft to
+         gripper base plate) -->
     <joint name="hand_tool_joint" type="fixed">
         <parent link="hand_link" />
         <child link="tool_link" />
-        <origin xyz="0 0 0.02" rpy="0 0 0" />
+        <origin xyz="0 0 0.01" rpy="0 0 0" />
     </joint>
 </robot>

File: src/robot_drive_by_moveit2/src/my_robot_description/urdf/gripper.xacro (robot description, xacro)
@@ -1,8 +1,27 @@
 <?xml version="1.0"?>
 <robot xmlns:xacro="http://www.ros.org/wiki/xacro">
+    <!-- ================================================================
+         Simplified parallel gripper.
+         Real hardware - 3D printed 2-finger gripper with a parallelogram
+         linkage driven by a sector gear from a ZP25S servo. Here it is
+         simplified to a prismatic (translating) 2-finger gripper, which is
+         accurate enough for planning and MuJoCo simulation.
+         Measured on the real gripper (metres) -
+           base plate   80 x 20 x 20 mm  (X width, Y depth, Z thickness)
+           finger       10 x 20 x 80 mm  (X thickness, Y depth, Z length)
+           grip length  100 mm from the base plate bottom face to the fingertip
+           opening      80 mm between the inner faces when fully open
+                        (symmetric, 40 mm travel per finger)
+         Joint convention -
+           master value 0.0    -> fully open  (80 mm gap)
+           master value 0.04   -> fully closed (0 mm gap)
+         ================================================================ -->
+    <!-- gripper_base_link - palm / base plate.
+         Origin sits on the mounting face at tool_link; the plate extends
+         +Z (away from the arm) by 20mm -->
     <link name="gripper_base_link">
         <visual>
             <geometry>
-                <box size="0.2 0.06 0.02" />
+                <box size="0.08 0.02 0.02" />
             </geometry>
             <origin xyz="0 0 0.01" rpy="0 0 0" />
@@ -11,13 +30,14 @@
         <collision>
             <geometry>
-                <box size="0.2 0.06 0.02" />
+                <box size="0.08 0.02 0.02" />
             </geometry>
             <origin xyz="0 0 0.01" rpy="0 0 0" />
         </collision>
     </link>
+    <!-- gripper_left_finger_link - finger plate, 80mm long along +Z -->
     <link name="gripper_left_finger_link">
         <visual>
             <geometry>
-                <box size="0.02 0.06 0.08" />
+                <box size="0.01 0.02 0.08" />
             </geometry>
             <origin xyz="0 0 0.04" rpy="0 0 0" />
@@ -26,13 +46,14 @@
         <collision>
             <geometry>
-                <box size="0.02 0.06 0.08" />
+                <box size="0.01 0.02 0.08" />
             </geometry>
             <origin xyz="0 0 0.04" rpy="0 0 0" />
         </collision>
     </link>
+    <!-- gripper_right_finger_link - mirror of the left finger -->
     <link name="gripper_right_finger_link">
         <visual>
             <geometry>
-                <box size="0.02 0.06 0.08" />
+                <box size="0.01 0.02 0.08" />
             </geometry>
             <origin xyz="0 0 0.04" rpy="0 0 0" />
@@ -41,23 +62,27 @@
         <collision>
             <geometry>
-                <box size="0.02 0.06 0.08" />
+                <box size="0.01 0.02 0.08" />
             </geometry>
             <origin xyz="0 0 0.04" rpy="0 0 0" />
         </collision>
     </link>
+    <!-- left finger joint - starts at the OPEN position (centre -45mm, inner
+         face -40mm) and travels +40mm in X to close -->
     <joint name="gripper_left_finger_joint" type="prismatic">
         <parent link="gripper_base_link" />
         <child link="gripper_left_finger_link" />
-        <origin xyz="-0.07 0 0.02" rpy="0 0 0" />
+        <origin xyz="-0.045 0 0.02" rpy="0 0 0" />
         <axis xyz="1 0 0" />
-        <limit effort="1000.0" velocity="1.0" lower="0.0" upper="0.06" />
+        <limit effort="100.0" velocity="0.5" lower="0.0" upper="0.04" />
     </joint>
+    <!-- right finger joint - mimic of the left one with multiplier -1, so it
+         moves the opposite way and keeps the gripper symmetric -->
     <joint name="gripper_right_finger_joint" type="prismatic">
         <parent link="gripper_base_link" />
         <child link="gripper_right_finger_link" />
-        <origin xyz="0.07 0 0.02" rpy="0 0 0" />
+        <origin xyz="0.045 0 0.02" rpy="0 0 0" />
         <axis xyz="1 0 0" />
         <mimic joint="gripper_left_finger_joint" multiplier="-1.0" />
-        <limit effort="1000.0" velocity="1.0" lower="-0.06" upper="0.0" />
+        <limit effort="100.0" velocity="0.5" lower="-0.04" upper="0.0" />
     </joint>
 </robot>
